File: charge_pcb/charge_pcb.kicad_pcb (KiCad board)
At the start: 2 copper layers, 31 parts, among them J1 PCB_1, J2 Battery, J3 Power Switch, J4 24V Out, J5 Motor_Left, J6 Motor_Cutter, J7 Motor_Right, Q1 BC547C, Q2 IRLML6344TRPBF, Q3 BC547C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

Commit message: Chargin Board changes
Parts:
- removed Logo: ESD-Logo_6.6x6mm_SilkScreen, Symbol:ESD-Logo_6.6x6mm_SilkScreen
- removed Logo2: OSHW-Logo2_7.3x6mm_SilkScreen, Symbol:OSHW-Logo2_7.3x6mm_SilkScreen
- added D6: Station LED, LED_THT:LED_D1.8mm_W3.3mm_H2.4mm, F.Cu at (88.6, 129.9)
- added R9: 4.7k, Resistor_THT:R_Axial_DIN0207_L6.3mm_D2.5mm_P7.62mm_Horizontal, F.Cu at (108.1, 120.8)
Routing:
- net Net-(D6-Pad2): track 0.00 -> 29.5 mm
- net GND: track 275.9 -> 284.4 mm
- net Net-(D2-Pad2): track 26.8 -> 29.6 mm
Other:
- board text added: "3.3V"

Commit message: Change Name of Mosfet
Parts:
- D6: value Station LED -> LED
- Q2, Q4: value IRLML6344TRPBF -> IRLB 8721
- R9: value 4.7k -> 4.7kO
Changed lines of the file:
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@@
       (effects (font (size 1 1) (thickness 0.15)))
     )
-    (fp_text value "Station LED" (at 1.53 4.61 90) (layer F.SilkS)
+    (fp_text value LED (at 1.53 4.61 90) (layer F.SilkS)
       (effects (font (size 0.7 0.7) (thickness 0.15)))
     )
@@
       (effects (font (size 1 1) (thickness 0.15)))
     )
-    (fp_text value 4.7k (at 3.81 2.37) (layer F.Fab)
+    (fp_text value 4.7kO (at 3.81 2.37) (layer F.Fab)
       (effects (font (size 1 1) (thickness 0.15)))
     )
@@
       (effects (font (size 1 1) (thickness 0.15)))
     )
-    (fp_text value IRLML6344TRPBF (at 2.286 1.9 90) (layer F.Fab)
+    (fp_text value "IRLB 8721" (at 2.286 1.9 90) (layer F.Fab)
       (effects (font (size 1 1) (thickness 0.15)))
     )
@@
       (effects (font (size 1 1) (thickness 0.15)))
     )
-    (fp_text value IRLML6344TRPBF (at 2.286 1.9) (layer F.Fab)
-      (effects (font (size 1 1) (thickness 0.15)))
-    )
+    (fp_text value "IRLB 8721" (at 2.286 1.9) (layer F.Fab)
+      (effects (font (size 1 1) (thickness 0.15)))
+    )

Commit message: Add Gerber Files
Parts:
- added H1: MountingHole_Pad, MountingHole:MountingHole_3.2mm_M3_DIN965_Pad_TopBottom, F.Cu at (73.1, 107.9)
- added H2: MountingHole_Pad, MountingHole:MountingHole_3.2mm_M3_DIN965_Pad_TopBottom, F.Cu at (179.6, 107.8)
- added H3: MountingHole_Pad, MountingHole:MountingHole_3.2mm_M3_DIN965_Pad_TopBottom, F.Cu at (179.7, 151.2)
- added H4: MountingHole_Pad, MountingHole:MountingHole_3.2mm_M3_DIN965_Pad_TopBottom, F.Cu at (73.2, 151.0)
Routing:
- net GND: track 284.4 -> 461.7 mm
