File: DUE_PCB/Ardumower.sch (KiCad schematic (older format))
At the start: 50 parts, among them J1 9V IN, J10 Sonar_R, J11 Sonar_C, J12 Sonar_L, J13 P_Right, J14 DS3231 RTC, J15 Button, J16 Button, J17 Button, J18 Button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

Commit message: File changes
Changed lines of the file:
@@
 F1 "file609243F3.sch" 50
 $EndSheet
+Wire Wire Line
+	2700 850  3550 850
+Wire Wire Line
+	3550 850  3550 5800
+Wire Wire Line
+	3550 5800 4850 5800
 $EndSCHEMATC
