File: DUE_PCB/Ardumower_2_firstroute.kicad_pcb (KiCad board)
At the start: 2 copper layers, 182.2 x 97.8 mm, 75 parts, among them J1 9V IN, J10 Sonar_R, J11 Sonar_C, J12 Sonar_L, J13 P_Right, J14 DS3231 RTC, J15 Button, J16 Button, J17 Button, J18 Button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

Commit message: File changes
Parts:
- removed D7: LED_24V, LED_THT:LED_D3.0mm
- removed D8: 1N5819, Diode_THT:D_DO-41_SOD81_P10.16mm_Horizontal
- removed J25: 24V IN, TerminalBlock:TerminalBlock_bornier-2_P5.08mm
- removed JP3: 24V, Connector_PinSocket_2.54mm:PinSocket_1x02_P2.54mm_Vertical
- removed R16: 1K5, Resistor_THT:R_Axial_DIN0207_L6.3mm_D2.5mm_P2.54mm_Vertical
- added REF**: Test-Point-Pin_Drill2.79mm, digikey-footprints:Test-Point-Pin_Drill2.79mm, F.Cu at (44.4, 39.2)
- added REF2: Test-Point-Pin_Drill2.79mm, digikey-footprints:Test-Point-Pin_Drill2.79mm, F.Cu at (44.6, 127.3)
- added REF3: Test-Point-Pin_Drill2.79mm, digikey-footprints:Test-Point-Pin_Drill2.79mm, F.Cu at (204.8, 126.8)
- added REF4: Test-Point-Pin_Drill2.79mm, digikey-footprints:Test-Point-Pin_Drill2.79mm, F.Cu at (204.8, 39.0)
- J1: value 9V IN -> Power 9-12V
- J16: value Button -> Button 1
- J17: value Button -> Button 2
- J18: value Button -> Button 3
- moved J16 118.8 mm to (98.6, 120.3)
- moved J6 118.6 mm to (46.8, 114.3)
- moved J7 118.6 mm to (54.7, 114.2)
- moved J20 103.9 mm to (46.8, 106.2), turned to 90 degrees
- moved J21 102.0 mm to (43.3, 87.8)
- moved U2 98.7 mm to (211.8, 133.3), turned to 90 degrees
- moved R26 87.3 mm to (187.5, 102.7)
- moved R25 73.9 mm to (187.6, 96.6)
- moved U1 67.3 mm to (211.8, 86.2), turned to 90 degrees
- moved R24 66.4 mm to (187.6, 89.7)
- moved JP6 56.8 mm to (193.9, 104.5)
- moved J19 55.5 mm to (139.0, 116.2)
- moved R23 54.9 mm to (187.4, 83.4)
- moved J18 51.7 mm to (106.6, 120.3)
- moved R22 46.7 mm to (187.4, 78.0)
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Routing:
- net GND: track 0.00 -> 785.4 mm
- net +9V: track 0.00 -> 80.5 mm
- net Net-(C1-Pad2): track 0.00 -> 22.2 mm
- net Net-(J1-Pad2): track 0.00 -> 8.95 mm
- net Net-(D1-Pad2): track 0.00 -> 5.48 mm
Other:
- board size 182.2 x 97.8 mm -> 169.3 x 96.8 mm
- board text added: "+"
- board text added: "GND"
- board text added: "RX2"
- board text added: "TX1"
- board text added: "TX2"
- board text added: "pinBatterySwitch"
- board text added: "pinChargeCurrent"
- board text added: "pinChargeRelay"
- board text added: "pinChargeVoltage"
- board text added: "pinVoltageMeasurement"
