File: DUE_PCB_V1.01/file609243F3.sch (KiCad schematic (older format))
At the start: 20 parts, among them J28 Motor Left, J29 Cutter Motor, J30 Motor Right, U1 MC33926, U2 MC33926

Commit message: first test
JP2 and JP3 redraw
Parts:
- U1, U2: symbol Lötpad_2,5mm:MC33926 -> Ardumower-rescue:MC33926-Lötpad_2,5mm
Changed lines of the file:
@@
 pinMotorRightPWM
 $Comp
-L Lötpad_2,5mm:MC33926 U?
+L Ardumower-rescue:MC33926-Lötpad_2,5mm U?
 U 1 1 60958C90
 P 3300 6450
@@
 $EndComp
 $Comp
-L Lötpad_2,5mm:MC33926 U?
+L Ardumower-rescue:MC33926-Lötpad_2,5mm U?
 U 1 1 60958C96
 P 3300 4300
