File: DUE_PCB_V1.01/_autosave-Ardumower.sch (KiCad schematic (older format))
At the start: 62 parts, among them J1 I2C_1, J10 Bumper Left, J11 Bumper Right, J12 P_Left, J13 P_Right, J14 Sonar_R, J15 Sonar_C, J16 Sonar_L, J17 US1, J18 US2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

Commit message: Update J30 and J32
Parts:
- added B1: SPARKFUN_LOGIC_LEVEL_CONVERTER, Boards:SPARKFUN_LOGIC_LEVEL_CONVERTER, symbol SparkFun-Boards:SPARKFUN_LOGIC_LEVEL_CONVERTER
- gave numbers to parts that had none: 4
Changed lines of the file:
@@
 	2700 5950 3100 5950
 $Comp
-L Device:R R?
+L Device:R R8
 U 1 1 609850CF
 P -950 4650
-F 0 "R?" V -1050 4650 50  0000 C CNN
+F 0 "R8" V -1050 4650 50  0000 C CNN
 F 1 "XXX" V -950 4650 50  0000 C CNN
 F 2 "Resistor_THT:R_Axial_DIN0207_L6.3mm_D2.5mm_P2.54mm_Vertical" V -1020 4650 50  0001 C CNN
@@
 $EndComp
 $Comp
-L Device:R R?
+L Device:R R13
 U 1 1 6098F377
 P -500 4650
-F 0 "R?" V -600 4650 50  0000 C CNN
+F 0 "R13" V -600 4650 50  0000 C CNN
 F 1 "XXX" V -500 4650 50  0000 C CNN
 F 2 "Resistor_THT:R_Axial_DIN0207_L6.3mm_D2.5mm_P2.54mm_Vertical" V -570 4650 50  0001 C CNN
@@
 SCL1
 $Comp
-L power:GND #PWR?
+L power:GND #PWR07
 U 1 1 609A6BE2
 P -150 6250
-F 0 "#PWR?" H -150 6000 50  0001 C CNN
+F 0 "#PWR07" H -150 6000 50  0001 C CNN
 F 1 "GND" V -145 6122 50  0000 R CNN
 F 2 "" H -150 6250 50  0001 C CNN
@@
 $EndComp
 $Comp
-L power:+3.3V #PWR?
+L power:+3.3V #PWR06
 U 1 1 609A6BEC
 P -1100 6000
-F 0 "#PWR?" H -1100 5850 50  0001 C CNN
+F 0 "#PWR06" H -1100 5850 50  0001 C CNN
 F 1 "+3.3V" V -1085 6128 50  0000 L CNN
 F 2 "" H -1100 6000 50  0001 C CNN
@@
 $EndComp
 $Comp
-L Device:R R?
+L Device:R R9
 U 1 1 609A6BF6
 P -950 6150
-F 0 "R?" V -1050 6150 50  0000 C CNN
+F 0 "R9" V -1050 6150 50  0000 C CNN
 F 1 "XXX" V -950 6150 50  0000 C CNN
 F 2 "Resistor_THT:R_Axial_DIN0207_L6.3mm_D2.5mm_P2.54mm_Vertical" V -1020 6150 50  0001 C CNN
@@
 $EndComp
 $Comp
-L Device:R R?
+L Device:R R27
 U 1 1 609A6C00
 P -500 6150
-F 0 "R?" V -600 6150 50  0000 C CNN
+F 0 "R27" V -600 6150 50  0000 C CNN
 F 1 "XXX" V -500 6150 50  0000 C CNN
 F 2 "Resistor_THT:R_Axial_DIN0207_L6.3mm_D2.5mm_P2.54mm_Vertical" V -570 6150 50  0001 C CNN
@@
 Wire Wire Line
 	-150 6000 -150 6150
+$Comp
+L SparkFun-Boards:SPARKFUN_LOGIC_LEVEL_CONVERTER B1
+U 1 1 609C0184
+P -700 2400
+F 0 "B1" H -700 3060 45  0000 C CNN
+F 1 "SPARKFUN_LOGIC_LEVEL_CONVERTER" H -700 2976 45  0000 C CNN
+F 2 "Boards:SPARKFUN_LOGIC_LEVEL_CONVERTER" H -700 2850 20  0001 C CNN
+F 3 "" H -700 2400 50  0001 C CNN
+F 4 "XXX-00000" H -700 2881 60  0000 C CNN "Field4"
+	1    -700 2400
+	1    0    0    -1
+$EndComp
 $EndSCHEMATC
