File: Charging_PCB/charge_pcb.kicad_pcb (KiCad board)
At the start: 2 copper layers, 35 parts, among them J1 PCB_1, J2 Battery, J3 Power Switch, J4 24V Out, J5 Motor_Left, J6 Motor_Cutter, J7 Motor_Right, Q1 BC547C, Q2 IRLB 8721, Q3 BC547C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

Commit message: PCB Changes
Parts:
- D6: value LED -> Station LED
- moved D5 41.6 mm to (129.1, 152.2), turned to 90 degrees
- moved J4 39.8 mm to (153.3, 148.5), turned to 180 degrees
- moved C1 39.8 mm to (121.1, 131.1), turned to 0 degrees
- moved J6 30.8 mm to (140.3, 148.4), turned to 180 degrees
- moved Q2 23.5 mm to (117.0, 130.0), turned to 180 degrees
- moved Q1 21.3 mm to (91.7, 130.0)
- moved R5 20.5 mm to (111.0, 145.8), turned to 0 degrees
- moved H3 18.9 mm to (160.8, 150.8)
- moved H2 18.8 mm to (160.8, 107.8)
- moved J2 18.3 mm to (135.4, 110.3)
- moved R3 18.1 mm to (97.8, 136.0), turned to 180 degrees
- moved D3 17.3 mm to (98.2, 124.1)
- moved Q4 17.2 mm to (145.8, 126.5), turned to 0 degrees
- moved R8 16.3 mm to (101.5, 140.8)
- moved D6 15.3 mm to (102.8, 124.0)
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Routing:
- net GND: track 461.7 -> 284.9 mm
- net pinChargeEnable: track 55.1 -> 19.5 mm
- net Net-(D6-Pad2): track 29.5 -> 5.10 mm
- net Net-(C1-Pad1): track 99.7 -> 121.6 mm
- net pinBatterySwitch: track 63.0 -> 41.2 mm
- net Net-(D2-Pad2): track 29.6 -> 50.1 mm
- net Net-(D3-Pad1): track 62.7 -> 43.8 mm
- net Net-(Q1-Pad1): track 26.3 -> 44.0 mm
- net pinChargeCurrent: track 76.7 -> 60.5 mm
- net pinBatteryVoltage: track 58.3 -> 44.4 mm
- net Net-(Q3-Pad2): track 7.20 -> 16.1 mm
- net Net-(D5-Pad2): track 45.4 -> 38.9 mm
- net Net-(Q3-Pad1): track 36.2 -> 42.4 mm
- net Net-(F2-Pad1): track 14.3 -> 20.3 mm
- net pinChargeVoltage: track 43.3 -> 46.2 mm
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Other:
- board outline added: 94.5 x 50.2 mm

Commit message: Small Changes
Change Q2 & Q4 to IRF9540N
Add Push Button to start the Due
Change pinChargeEnable to pinChargeRelay
Parts:
- added SW1: SW_Push, Connector_JST:JST_XH_B2B-XH-A_1x02_P2.50mm_Vertical, F.Cu at (139.5, 163.1)
- D6: value Station LED -> LED
- Q2, Q4: value IRLB 8721 -> IRF9540N; footprint Package_TO_SOT_THT:SIPAK-1EP_Horizontal_TabDown -> Package_TO_SOT_THT:TO-220-3_Vertical
- moved Q4 49.8 mm to (118.7, 168.4)
- moved Q2 32.5 mm to (118.7, 162.4), turned to 0 degrees
Connections:
- net pinChargeEnable renamed pinChargeRelay
- J1 pad 6: pinVoltageMeasurement -> (no net)
- Q2 pad 2: Net-(D3-Pad1) -> Net-(D2-Pad2)
- Q2 pad 3: Net-(D2-Pad2) -> Net-(D3-Pad1)
- Q4 pad 2: Net-(C1-Pad1) -> Net-(D5-Pad2)
- Q4 pad 3: Net-(D5-Pad2) -> Net-(C1-Pad1)
- U1 pad 1: +3V3 -> pinBatterySwitch

Commit message: Only placeholder
Parts:
- moved Q4 44.0 mm to (145.2, 133.3)
- moved Q2 25.8 mm to (117.2, 136.6), turned to 180 degrees
- moved J1 10.7 mm to (69.3, 131.2), turned to 0 degrees
- moved SW1 6.16 mm to (134.2, 159.9)
Changed lines of the file:
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@@
   )
   (module Connector_JST:JST_XH_B2B-XH-A_1x02_P2.50mm_Vertical (layer F.Cu)
-    (at 139.47 163.1)
+    (at 134.21 159.89)
     (descr "JST XH series connector, B2B-XH-A (http://www.jst-mfg.com/product/pdf/eng/eXH.pdf), generated with kicad-footprint-generator")
     (tags "connector JST XH vertical")
@@
   )
   (module Package_TO_SOT_THT:TO-220-3_Vertical (layer F.Cu)
-    (at 118.72 168.37)
+    (at 145.21 133.27)
     (descr "TO-220-3, Vertical, RM 2.54mm, see https://www.vishay.com/docs/66542/to-220-1.pdf")
     (tags "TO-220-3 Vertical RM 2.54mm")
@@
   )
   (module Package_TO_SOT_THT:TO-220-3_Vertical (layer F.Cu)
-    (at 118.72 162.41)
+    (at 117.23 136.64 180)
     (descr "TO-220-3, Vertical, RM 2.54mm, see https://www.vishay.com/docs/66542/to-220-1.pdf")
     (tags "TO-220-3 Vertical RM 2.54mm")
@@
     (fp_line (start 7.79 1.51) (end 7.79 -3.4) (layer F.CrtYd) (width 0.05))
     (fp_line (start 7.79 -3.4) (end -2.71 -3.4) (layer F.CrtYd) (width 0.05))
-    (pad 3 thru_hole oval (at 5.08 0) (size 1.905 2) (drill 1.1) (layers *.Cu *.Mask)
+    (pad 3 thru_hole oval (at 5.08 0 180) (size 1.905 2) (drill 1.1) (layers *.Cu *.Mask)
       (net 6 "Net-(D3-Pad1)"))
-    (pad 2 thru_hole oval (at 2.54 0) (size 1.905 2) (drill 1.1) (layers *.Cu *.Mask)
+    (pad 2 thru_hole oval (at 2.54 0 180) (size 1.905 2) (drill 1.1) (layers *.Cu *.Mask)
       (net 5 "Net-(D2-Pad2)"))
-    (pad 1 thru_hole rect (at 0 0) (size 1.905 2) (drill 1.1) (layers *.Cu *.Mask)
+    (pad 1 thru_hole rect (at 0 0 180) (size 1.905 2) (drill 1.1) (layers *.Cu *.Mask)
       (net 15 "Net-(Q1-Pad1)"))
     (model ${KISYS3DMOD}/Package_TO_SOT_THT.3dshapes/TO-220-3_Vertical.wrl
@@
   )
   (module Connector_PinHeader_2.54mm:PinHeader_1x06_P2.54mm_Vertical (layer F.Cu)
-    (at 72.72 141.33 180)
+    (at 69.27 131.25)
     (descr "Through hole straight pin header, 1x06, 2.54mm pitch, single row")
     (tags "Through hole pin header THT 1x06 2.54mm single row")
@@
       (effects (font (size 1 1) (thickness 0.15)))
     )
-    (pad 6 thru_hole oval (at 0 12.7 180) (size 1.7 1.7) (drill 1) (layers *.Cu *.Mask))
-    (pad 5 thru_hole oval (at 0 10.16 180) (size 1.7 1.7) (drill 1) (layers *.Cu *.Mask)
+    (pad 6 thru_hole oval (at 0 12.7) (size 1.7 1.7) (drill 1) (layers *.Cu *.Mask))
+    (pad 5 thru_hole oval (at 0 10.16) (size 1.7 1.7) (drill 1) (layers *.Cu *.Mask)
       (net 20 pinChargeRelay))
-    (pad 4 thru_hole oval (at 0 7.62 180) (size 1.7 1.7) (drill 1) (layers *.Cu *.Mask)
+    (pad 4 thru_hole oval (at 0 7.62) (size 1.7 1.7) (drill 1) (layers *.Cu *.Mask)
       (net 10 pinChargeCurrent))
-    (pad 3 thru_hole oval (at 0 5.08 180) (size 1.7 1.7) (drill 1) (layers *.Cu *.Mask)
+    (pad 3 thru_hole oval (at 0 5.08) (size 1.7 1.7) (drill 1) (layers *.Cu *.Mask)
       (net 11 pinChargeVoltage))
-    (pad 2 thru_hole oval (at 0 2.54 180) (size 1.7 1.7) (drill 1) (layers *.Cu *.Mask)
+    (pad 2 thru_hole oval (at 0 2.54) (size 1.7 1.7) (drill 1) (layers *.Cu *.Mask)
       (net 12 pinBatterySwitch))
-    (pad 1 thru_hole rect (at 0 0 180) (size 1.7 1.7) (drill 1) (layers *.Cu *.Mask)
+    (pad 1 thru_hole rect (at 0 0) (size 1.7 1.7) (drill 1) (layers *.Cu *.Mask)
       (net 13 pinBatteryVoltage))
     (model ${KISYS3DMOD}/Connector_PinHeader_2.54mm.3dshapes/PinHeader_1x06_P2.54mm_Vertical.wrl

Commit message: Improve Q2 and Q4
Parts:
- moved Q2 6.97 mm to (117.4, 129.7)
- moved Q4 6.91 mm to (145.5, 126.4)
Connections:
- Q2 pad 2: Net-(D2-Pad2) -> Net-(D3-Pad1)
- Q2 pad 3: Net-(D3-Pad1) -> Net-(D2-Pad2)
- Q4 pad 2: Net-(D5-Pad2) -> Net-(C1-Pad1)
- Q4 pad 3: Net-(C1-Pad1) -> Net-(D5-Pad2)

Commit message: Add Bernards Changes
Parts:
- removed J2: Battery, TerminalBlock:TerminalBlock_bornier-2_P5.08mm
- removed J3: Power Switch, TerminalBlock:TerminalBlock_bornier-2_P5.08mm
- removed J4: 24V Out, TerminalBlock:TerminalBlock_bornier-2_P5.08mm
- removed J5: Motor_Left, TerminalBlock:TerminalBlock_bornier-2_P5.08mm
- removed J6: Motor_Cutter, TerminalBlock:TerminalBlock_bornier-2_P5.08mm
- removed J7: Motor_Right, TerminalBlock:TerminalBlock_bornier-2_P5.08mm
- removed SW1: SW_Push, Connector_JST:JST_XH_B2B-XH-A_1x02_P2.50mm_Vertical
- added  J6 Motor: Motor_Cutter, TerminalBlock:TerminalBlock_bornier-2_P5.08mm, F.Cu at (160.0, 130.8)
- added D8: SB1240, Diode_THT:D_DO-41_SOD81_P10.16mm_Horizontal, F.Cu at (130.8, 129.5)
- added J2 Bat +: Battery, TerminalBlock:TerminalBlock_bornier-2_P5.08mm, F.Cu at (139.7, 109.2)
- added J3 Switch: Power Switch, TerminalBlock:TerminalBlock_bornier-2_P5.08mm, F.Cu at (151.1, 109.2)
- added J4 Out: 24V Out, TerminalBlock:TerminalBlock_bornier-2_P5.08mm, F.Cu at (137.2, 149.9)
- added J5 Motor: Motor_Drive, TerminalBlock:TerminalBlock_bornier-2_P5.08mm, F.Cu at (160.0, 118.1)
- added J7 Out: 24V Out, TerminalBlock:TerminalBlock_bornier-2_P5.08mm, F.Cu at (125.7, 149.9)
- added J8: Start, Connector_JST:JST_XH_B2B-XH-A_1x02_P2.50mm_Vertical, F.Cu at (114.3, 149.9)
- added J9 Out: 24V out, TerminalBlock:TerminalBlock_bornier-2_P5.08mm, F.Cu at (148.6, 149.9)
- added R10: 2k2, Resistor_THT:R_Axial_DIN0207_L6.3mm_D2.5mm_P7.62mm_Horizontal, F.Cu at (96.5, 144.8)
- added R11: 2k2, Resistor_THT:R_Axial_DIN0207_L6.3mm_D2.5mm_P7.62mm_Horizontal, F.Cu at (91.4, 128.3)
- J1: footprint Connector_PinHeader_2.54mm:PinHeader_1x06_P2.54mm_Vertical -> Connector_JST:JST_XH_B6B-XH-A_1x06_P2.50mm_Vertical
- U1: value ACS712 -> INA169
- moved Q3 26.7 mm to (146.1, 120.7)
- moved Q2 20.2 mm to (97.8, 134.6), turned to 90 degrees
- moved D5 18.2 mm to (124.5, 134.6), turned to 180 degrees
- moved C1 14.7 mm to (109.2, 139.7)
- moved Q4 11.8 mm to (134.6, 121.9)
- moved Q1 11.7 mm to (80.0, 130.8)
- moved R2 10.9 mm to (115.6, 129.5), turned to 0 degrees
- moved R5 10.7 mm to (100.3, 145.8)
- moved R7 10.5 mm to (108.0, 151.1)
- moved J1 10.2 mm to (72.4, 141.0), turned to 90 degrees
- moved R4 10.2 mm to (87.6, 141.0)
- moved R3 10.2 mm to (87.6, 136.0)
- moved F2 9.60 mm to (139.7, 138.4), turned to 180 degrees
- moved R8 8.78 mm to (92.7, 141.0)
- moved R6 7.62 mm to (115.6, 142.2), turned to 0 degrees
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Connections:
- net pinChargeRelay renamed pinChargeEnable
- J1 pad 6: (no net) -> +3V3
- Q2 pad 2: Net-(D3-Pad1) -> Net-(D2-Pad2)
- Q2 pad 3: Net-(D2-Pad2) -> Net-(D3-Pad1)
- Q4 pad 2: Net-(C1-Pad1) -> Net-(D5-Pad2)
- Q4 pad 3: Net-(D5-Pad2) -> Net-(C1-Pad1)
- R1 pad 1: Net-(D2-Pad2) -> Net-(D1-Pad1)
- R9 pad 1: Net-(D2-Pad2) -> Net-(D1-Pad1)
- U1 pad 1: pinBatterySwitch -> +3V3
Routing:
- net GND: track 284.9 -> 346.3 mm
- net +3V3: track 0.00 -> 44.4 mm
- net Net-(D8-Pad2): track 0.00 -> 36.4 mm
- net Net-(Q3-Pad2): track 16.1 -> 51.1 mm
- net Net-(D1-Pad1): track 29.3 -> 55.9 mm
- net Net-(C1-Pad1): track 121.6 -> 99.8 mm
- net Net-(D2-Pad2): track 50.1 -> 34.4 mm
- net Net-(Q1-Pad1): track 44.0 -> 29.5 mm
- net Net-(F2-Pad1): track 20.3 -> 33.5 mm
- net pinChargeEnable: track 19.5 -> 30.6 mm
- net pinBatteryVoltage: track 44.4 -> 34.3 mm
- net pinBatterySwitch: track 41.2 -> 31.7 mm
- net Net-(J8-Pad1): track 42.4 -> 51.6 mm
- net Net-(J2-Pad1): track 45.8 -> 50.8 mm
- net Net-(D3-Pad1): track 43.8 -> 47.1 mm
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Other:
- board size 94.5 x 50.2 mm -> 96.5 x 50.8 mm
- board text added: "GND"
- board text added: "PowerBoard by S.D/B.B V1.01"
- board text removed: "Mower Charging Board by S.D V1.0"
- board text removed: "VoltageMeasurement"
