File: Charging_PCB/charge_pcb.kicad_sch (KiCad schematic)
At the start: 40 parts, among them J1 PCB_1, J2 Battery, J3 Power Switch, J4 24V Out, J5 Motor_Drive, J6 Motor_Cutter, J7 24V Out, J8 Start, J9 24V out, Q1 BC547C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

Commit message: Add Schematic PDF and new Picture
Other:
- moved on the sheet: Q4
Changed lines of the file:
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@@
   (junction (at 201.93 79.375) (diameter 0.9144) (color 0 0 0 0))
   (junction (at 201.93 93.98) (diameter 0.9144) (color 0 0 0 0))
+  (junction (at 217.17 66.04) (diameter 0.9144) (color 0 0 0 0))
   (junction (at 217.297 66.04) (diameter 0.9144) (color 0 0 0 0))
-  (junction (at 225.425 46.99) (diameter 0.9144) (color 0 0 0 0))
-  (junction (at 225.425 57.15) (diameter 0.9144) (color 0 0 0 0))
   (junction (at 234.95 57.15) (diameter 0.9144) (color 0 0 0 0))
   (junction (at 234.95 73.66) (diameter 0.9144) (color 0 0 0 0))
@@
     (stroke (width 0) (type solid) (color 0 0 0 0))
   )
-  (wire (pts (xy 201.93 66.04) (xy 217.297 66.04))
+  (wire (pts (xy 201.93 66.04) (xy 217.17 66.04))
     (stroke (width 0) (type solid) (color 0 0 0 0))
   )
@@
     (stroke (width 0) (type solid) (color 0 0 0 0))
   )
+  (wire (pts (xy 217.17 52.07) (xy 217.17 66.04))
+    (stroke (width 0) (type solid) (color 0 0 0 0))
+  )
+  (wire (pts (xy 217.17 66.04) (xy 217.297 66.04))
+    (stroke (width 0) (type solid) (color 0 0 0 0))
+  )
   (wire (pts (xy 217.297 52.07) (xy 217.297 66.04))
     (stroke (width 0) (type solid) (color 0 0 0 0))
@@
     (stroke (width 0) (type solid) (color 0 0 0 0))
   )
-  (wire (pts (xy 224.79 46.99) (xy 225.425 46.99))
-    (stroke (width 0) (type solid) (color 0 0 0 0))
-  )
-  (wire (pts (xy 224.79 57.15) (xy 225.425 57.15))
-    (stroke (width 0) (type solid) (color 0 0 0 0))
-  )
-  (wire (pts (xy 225.425 46.99) (xy 234.95 46.99))
-    (stroke (width 0) (type solid) (color 0 0 0 0))
-  )
-  (wire (pts (xy 225.425 57.15) (xy 229.87 57.15))
+  (wire (pts (xy 224.79 46.99) (xy 234.95 46.99))
+    (stroke (width 0) (type solid) (color 0 0 0 0))
+  )
+  (wire (pts (xy 224.79 57.15) (xy 229.87 57.15))
     (stroke (width 0) (type solid) (color 0 0 0 0))
   )
@@
     (pin "3")
   )
-  (symbol (lib_id "Transistor_FET:IRF9540N") (at 222.885 52.07 0) (unit 1)
-    (in_bom yes) (on_board yes)
-    (property "Reference" "Q4" (id 0) (at 228.0666 50.9016 0)
-      (effects (font (size 1.27 1.27)) (justify left))
-    )
-    (property "Value" "IRF9540N" (id 1) (at 228.0666 53.213 0)
-      (effects (font (size 1.27 1.27)) (justify left))
-    )
-    (property "Footprint" "Package_TO_SOT_THT:TO-220-3_Vertical" (id 2) (at 227.965 53.975 0)
+  (symbol (lib_id "Transistor_FET:IRF9540N") (at 222.25 52.07 0) (unit 1)
+    (in_bom yes) (on_board yes)
+    (property "Reference" "Q4" (id 0) (at 227.4316 50.9016 0)
+      (effects (font (size 1.27 1.27)) (justify left))
+    )
+    (property "Value" "IRF9540N" (id 1) (at 227.4316 53.213 0)
+      (effects (font (size 1.27 1.27)) (justify left))
+    )
+    (property "Footprint" "Package_TO_SOT_THT:TO-220-3_Vertical" (id 2) (at 227.33 53.975 0)
       (effects (font (size 1.27 1.27) italic) (justify left) hide)
     )
-    (property "Datasheet" "http://www.irf.com/product-info/datasheets/data/irf9540n.pdf" (id 3) (at 222.885 52.07 0)
+    (property "Datasheet" "http://www.irf.com/product-info/datasheets/data/irf9540n.pdf" (id 3) (at 222.25 52.07 0)
       (effects (font (size 1.27 1.27)) (justify left) hide)
     )

Commit message: Small changes
Changed lines of the file:
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@@
   (junction (at 201.93 93.98) (diameter 0.9144) (color 0 0 0 0))
   (junction (at 217.17 66.04) (diameter 0.9144) (color 0 0 0 0))
-  (junction (at 217.297 66.04) (diameter 0.9144) (color 0 0 0 0))
   (junction (at 234.95 57.15) (diameter 0.9144) (color 0 0 0 0))
   (junction (at 234.95 73.66) (diameter 0.9144) (color 0 0 0 0))
@@
     (stroke (width 0) (type solid) (color 0 0 0 0))
   )
-  (wire (pts (xy 217.297 52.07) (xy 217.297 66.04))
-    (stroke (width 0) (type solid) (color 0 0 0 0))
-  )
   (wire (pts (xy 217.297 66.04) (xy 217.297 79.375))
     (stroke (width 0) (type solid) (color 0 0 0 0))
   )
-  (wire (pts (xy 217.805 52.07) (xy 217.297 52.07))
-    (stroke (width 0) (type solid) (color 0 0 0 0))
-  )
